Commit message: randomize room and start orientation

File: hamstir_gym/data/room2x12.urdf (robot description, URDF)
Before this commit: robot room, 6 links, 5 joints
Links:
- removed link center_link
- link east_link: mass 24300 -> 972; geometry collision box size=12 0.01 3; visual box size=12 0.01 3
- link floor_link: mass 48600 -> 3888; geometry collision box size=12 12 0.01; visual box size=12 12 0.01
- link north_link: mass 24300 -> 162; geometry collision box size=2 0.01 3; visual box size=2 0.01 3
- link south_link: mass 24300 -> 162; geometry collision box size=2 0.01 3; visual box size=2 0.01 3
- link west_link: mass 24300 -> 972; geometry collision box size=12 0.01 3; visual box size=12 0.01 3
Joints:
- removed joint center_joint
- joint east_joint: origin xyz=3 0 0 rpy=0 0 0 -> xyz=1 0 0 rpy=0 0 0
- joint north_joint: origin xyz=0 3 0 rpy=0 0 0 -> xyz=0 6 0 rpy=0 0 0
- joint south_joint: origin xyz=0 -3 0 rpy=0 0 0 -> xyz=0 -6 0 rpy=0 0 0
- joint west_joint: origin xyz=-3 0 0 rpy=0 0 0 -> xyz=-1 0 0 rpy=0 0 0
