Commit message: change gibson train to allenville

File: hamstir_gym/data/tb_base.urdf (robot description, URDF)
Before this commit: robot turtlebot, 7 links, 6 joints
Joints:
- joint eye_joint: origin xyz=0 0.05 0 rpy=1.57079632679 0 -1.57079632679 -> xyz=0 0.05 0.1 rpy=1.57079632679 0 -1.57079632679
