Commit message: allow different image dimensions in gym env

File: hamstir_gym/data/room12x12.urdf (robot description, URDF)
Before this commit: robot room12x12, 9 links, 8 joints
Links:
- added link ceiling_link, mass 3888; collision box size=12 12 0.01; visual box size=12 12 0.01
Joints:
- added joint ceiling_joint: type fixed, parent floor_link, child ceiling_link
