Commit message: full resetSimulation on episode reset

File: hamstir_gym/data/car.urdf (robot description, URDF)
Before this commit: robot car, 6 links, 5 joints
Links:
- link base_link: geometry collision cylinder length=0.10938 radius=0.1; visual cylinder length=0.10938 radius=0.1
- link camera_link: mass 0.1 -> 0.009; geometry collision box size=0.01 0.03 0.03; visual box size=0.01 0.03 0.03
Joints:
- joint camera_joint: origin xyz=0.18 0 0.06 rpy=0 0 0 -> xyz=0.06 0 0.1 rpy=0 0 0
- joint caster_back_joint: origin xyz=-0.135 0 0.009 rpy=-1.570796327 0 0 -> xyz=-0.05 0 0.009 rpy=-1.570796327 0 0
- joint caster_front_joint: origin xyz=0.115 0 0.007 rpy=-1.570796327 0 0 -> xyz=0.05 0 0.007 rpy=-1.570796327 0 0
- joint left_wheel_joint: origin xyz=0 0.115 0.025 rpy=-1.570796327 0 0 -> xyz=0 0.06 0.025 rpy=-1.570796327 0 0
- joint right_wheel_joint: origin xyz=0 -0.115 0.025 rpy=-1.570796327 0 0 -> xyz=0 -0.06 0.025 rpy=-1.570796327 0 0

Commit message: update model for gibson

File: hamstir_gym/data/car.urdf (robot description, URDF)
Before this commit: robot car, 6 links, 5 joints
Links:
- removed link camera_link
- added link eyes, mass 0.009; collision box size=0.01 0.03 0.03; visual box size=0.01 0.03 0.03
Joints:
- removed joint camera_joint
- added joint eyes_joint: type fixed, parent base_link, child eyes, origin xyz=0.06 0 0.1 rpy=0 0 0

Commit message: add larger wall buffer

File: hamstir_gym/data/car.urdf (robot description, URDF)
Before this commit: robot car, 6 links, 5 joints
Links:
- link eyes: geometry collision box size=0.01 0.03 0.03; visual box size=0.001 0.003 0.003
Joints:
- joint eyes_joint: origin xyz=0.06 0 0.1 rpy=0 0 0 -> xyz=0.05 0 0.1 rpy=0 0 0

Commit message: fix raspi camera fov

File: hamstir_gym/data/car.urdf (robot description, URDF)
Before this commit: robot car, 6 links, 5 joints
Joints:
- joint eyes_joint: origin xyz=0.05 0 0.1 rpy=0 0 0 -> xyz=0.06 0 0.1 rpy=0 0 0
